Commit message: Fixed gravity and cost function

File: robots/ur_description/urdf/ur16e.urdf (robot description, URDF)
Before this commit: robot ur16e_robot, 11 links, 10 joints
Links:
- link tool0: geometry collision cylinder length=0.12 radius=0.01; visual cylinder length=0.12 radius=0.01
Joints:
- joint base_link-base_link_inertia: origin xyz=0 0 0 rpy=0 0 3.141592653589793 -> xyz=0 0 0 rpy=0 0 1.5708

Commit message: New sim example and updated real robot example

File: robots/ur_description/urdf/ur16e.urdf (robot description, URDF)
Before this commit: robot ur16e_robot, 11 links, 10 joints
Links:
- link tool0: geometry collision cylinder length=0.115 radius=0.01; visual cylinder length=0.115 radius=0.01
