Commit message: Extend EEF to 0.20 m; derive TCP offset from URDF
- URDF tool0 cylinder: 0.115 → 0.20 m (length, center Z, TCP sphere, inertia CoM)
- Add get_tool_length() to ur16e.py: parses the collision cylinder as the single
  source of truth so planner and visualiser always match the physical geometry
- planner.py: remove hardcoded TCP_OFFSET_LOCAL=0.115; __init__ calls get_tool_length()
- world.py: replace hardcoded 0.12 (had a 5 mm mismatch) with get_tool_length()

Co-Authored-By: Claude Sonnet 4.6 <noreply@anthropic.com>

File: assets/robots/ur_description/urdf/ur16e.urdf (robot description, URDF)
Before this commit: robot ur16e_robot, 11 links, 10 joints
Links:
- link tool0: geometry collision cylinder length=0.20 radius=0.01; visual cylinder length=0.20 radius=0.01
