Commit message: Real robot running!

File: assets/robots/ur_description/urdf/ur16e.urdf (robot description, URDF)
Before this commit: robot ur16e_robot, 11 links, 10 joints
Links:
- link tool0: geometry collision cylinder length=0.12 radius=0.0025; visual cylinder length=0.12 radius=0.0025

Commit message: merge

File: assets/robots/ur_description/urdf/ur16e.urdf (robot description, URDF)
Before this commit: robot ur16e_robot, 11 links, 10 joints
Links:
- link tool0: geometry collision cylinder length=0.115 radius=0.0025; collision sphere radius=0.005

Commit message: pipeline testing MCTS -> robot working

File: assets/robots/ur_description/urdf/ur16e.urdf (robot description, URDF)
Before this commit: robot ur16e_robot, 11 links, 10 joints
Links:
- link tool0: geometry collision cylinder length=0.13 radius=0.0025; collision sphere radius=0.005
