Commit message: Working on real robot with modsd

File: assets/robots/ur_description/urdf/ur16e.urdf (robot description, URDF)
Before this commit: robot ur16e_robot, 11 links, 10 joints
Links:
- link tool0: geometry collision cylinder length=0.034 radius=0.04; collision cylinder length=0.096 radius=0.0025
